File: eve-flight-computer.kicad_pcb (KiCad board)
At the start: 6 copper layers, 0 parts

Commit message: Rev. 1
Parts:
- added BT1: ML414H, kicad-egglib:ML414H, F.Cu at (116.5, 55.5)
- added C1: 4.7uF, kicad-egglib:0402_1005M, B.Cu at (140.5, 85.0)
- added C10: 100nF, kicad-egglib:0402_1005M, B.Cu at (138.2, 71.8)
- added C11: 100nF, kicad-egglib:0402_1005M, B.Cu at (138.2, 65.2)
- added C12: 100nF, kicad-egglib:0402_1005M, B.Cu at (127.8, 60.8)
- added C13: 100nF, kicad-egglib:0402_1005M, B.Cu at (121.2, 60.8)
- added C14: 100nF, kicad-egglib:0402_1005M, B.Cu at (132.8, 60.8)
- added C15: 100nF, kicad-egglib:0402_1005M, B.Cu at (116.8, 81.2)
- added C16: 2.2uF, kicad-egglib:0402_1005M, B.Cu at (137.8, 82.2)
- added C17: 100nF, kicad-egglib:0402_1005M, F.Cu at (143.8, 56.0)
- added C18: 2.2uF, kicad-egglib:0402_1005M, B.Cu at (138.2, 66.2)
- added C19: 10uF, kicad-egglib:0805_2012M, B.Cu at (147.8, 70.2)
- added C2: 100nF, kicad-egglib:0402_1005M, B.Cu at (116.8, 67.8)
- added C20: 47uF, Capacitor_SMD:C_1206_3216Metric, B.Cu at (147.0, 65.0)
- added C21: 100nF, kicad-egglib:0402_1005M, B.Cu at (106.5, 59.8)
- added C22: 100nF, kicad-egglib:0402_1005M, B.Cu at (107.5, 59.8)
- added C23: 100nF, kicad-egglib:0402_1005M, B.Cu at (105.2, 56.5)
- added C24: 100nF, kicad-egglib:0402_1005M, B.Cu at (105.2, 57.5)
- added C25: 100nF, kicad-egglib:0402_1005M, F.Cu at (112.5, 57.0)
- added C26: 4.7uF, kicad-egglib:0402_1005M, F.Cu at (112.5, 59.0)
- added C27: 100nF, kicad-egglib:0402_1005M, B.Cu at (121.8, 95.5)
- added C28: 100nF, kicad-egglib:0402_1005M, B.Cu at (127.8, 94.0)
- added C29: 100nF, kicad-egglib:0402_1005M, B.Cu at (128.2, 103.0)
- added C3: 100nF, kicad-egglib:0402_1005M, B.Cu at (116.8, 73.2)
- added C30: 100nF, kicad-egglib:0402_1005M, B.Cu at (124.5, 105.2)
- added C31: 100nF, kicad-egglib:0402_1005M, B.Cu at (125.5, 105.2)
- added C32: 10uF, kicad-egglib:0805_2012M, F.Cu at (107.5, 114.0)
- added C33: 100nF, kicad-egglib:0402_1005M, F.Cu at (124.0, 47.0)
- added C34: 100nF, kicad-egglib:0402_1005M, B.Cu at (124.2, 67.0)
- added C35: 10uF, kicad-egglib:0805_2012M, F.Cu at (131.0, 131.5)
- added C36: 100nF, kicad-egglib:0402_1005M, B.Cu at (117.2, 94.0)
- added C37: 100nF, kicad-egglib:0402_1005M, B.Cu at (124.2, 75.0)
- added C38: 47uF, Capacitor_SMD:C_1206_3216Metric, B.Cu at (103.5, 65.0)
- added C39: 47uF, Capacitor_SMD:C_1206_3216Metric, B.Cu at (103.5, 70.0)
- added C4: 100nF, kicad-egglib:0402_1005M, B.Cu at (116.8, 79.8)
- added C40: 47uF, Capacitor_SMD:C_1206_3216Metric, B.Cu at (103.5, 75.0)
- added C41: 47uF, Capacitor_SMD:C_1206_3216Metric, B.Cu at (103.5, 80.0)
- added C42: 100nF, kicad-egglib:0402_1005M, F.Cu at (115.5, 111.0)
- added C43: 10uF, kicad-egglib:0805_2012M, F.Cu at (139.2, 101.2)
- added C44: 10uF, kicad-egglib:0805_2012M, F.Cu at (152.0, 97.0)
- added C45: 10uF, kicad-egglib:0805_2012M, F.Cu at (116.0, 105.0)
- added C46: 47uF, Capacitor_SMD:C_1206_3216Metric, B.Cu at (144.0, 107.0)
- added C47: 47uF, Capacitor_SMD:C_1206_3216Metric, B.Cu at (144.0, 112.0)
- added C48: 47uF, Capacitor_SMD:C_1206_3216Metric, B.Cu at (144.0, 117.0)
- added C49: 47uF, Capacitor_SMD:C_1206_3216Metric, B.Cu at (144.0, 122.0)
- added C5: 100nF, kicad-egglib:0402_1005M, B.Cu at (122.8, 82.8)
- added C50: 47uF, Capacitor_SMD:C_1206_3216Metric, B.Cu at (144.0, 127.0)
- added C51: 47uF, Capacitor_SMD:C_1206_3216Metric, B.Cu at (144.0, 132.0)
- added C52: 22uF, kicad-egglib:0805_2012M, F.Cu at (121.5, 111.0)
- added C53: 22uF, kicad-egglib:0805_2012M, F.Cu at (121.5, 113.0)
- added C54: 100nF, kicad-egglib:0402_1005M, F.Cu at (112.5, 86.2)
- added C6: 100nF, kicad-egglib:0402_1005M, B.Cu at (128.8, 82.2)
- added C7: 100nF, kicad-egglib:0402_1005M, B.Cu at (133.8, 82.2)
- added C8: 100nF, kicad-egglib:0402_1005M, B.Cu at (138.8, 82.2)
- added C9: 100nF, kicad-egglib:0402_1005M, B.Cu at (138.2, 77.2)
- added D1: Red, Diode_SMD:D_0603_1608Metric, F.Cu at (142.0, 95.0)
- added D10: 11V, Diode_SMD:D_SOD-123, B.Cu at (103.5, 77.5)
- added D11: 11V, Diode_SMD:D_SOD-123, B.Cu at (103.5, 82.5)
- added D2: Green, Diode_SMD:D_0603_1608Metric, F.Cu at (142.0, 93.5)
- added D3: Blue, Diode_SMD:D_0603_1608Metric, F.Cu at (142.0, 92.0)
- added D4: Yellow, Diode_SMD:D_0603_1608Metric, F.Cu at (142.0, 90.5)
- added D5: PMEG4005EJ, Diode_SMD:D_SOD-323, F.Cu at (116.5, 60.0)
- added D6: 11V, Diode_SMD:D_SOD-123, B.Cu at (103.5, 67.5)
- added D7: UPS115UE3, Diode_SMD:D_Powermite_AK, F.Cu at (117.0, 101.0)
- added D8: UPS115UE3, Diode_SMD:D_Powermite_AK, F.Cu at (113.0, 102.0)
- added D9: 11V, Diode_SMD:D_SOD-123, B.Cu at (103.5, 72.5)
- added J1: USB4110, Connector_USB:USB_C_Receptacle_GCT_USB4110, F.Cu at (138.0, 48.7)
- added J10: SERVO, Connector_PinHeader_2.54mm:PinHeader_1x03_P2.54mm_Vertical, F.Cu at (153.0, 122.0)
- added J11: SERVO, Connector_PinHeader_2.54mm:PinHeader_1x03_P2.54mm_Vertical, F.Cu at (153.0, 117.0)
- added J12: PYRO, Connector_PinSocket_2.54mm:PinSocket_1x12_P2.54mm_Vertical, F.Cu at (99.0, 65.0)
- added J13: SERVO, Connector_PinHeader_2.54mm:PinHeader_1x03_P2.54mm_Vertical, F.Cu at (153.0, 112.0)
- added J14: SERVO, Connector_PinHeader_2.54mm:PinHeader_1x03_P2.54mm_Vertical, F.Cu at (153.0, 107.0)
- added J2: ARM Cortex Debug, Connector_PinHeader_1.27mm:PinHeader_2x05_P1.27mm_Vertical_SMD, F.Cu at (149.0, 58.0)
- added J3: GPIO, Connector_PinSocket_2.54mm:PinSocket_1x12_P2.54mm_Vertical, F.Cu at (151.0, 65.0)
- added J4: SMA, Connector_Coaxial:SMA_Amphenol_132289_EdgeMount, F.Cu at (111.0, 48.4)
- added J5: SMA, Connector_Coaxial:SMA_Amphenol_132289_EdgeMount, B.Cu at (98.4, 122.0)
- added J6: SMA, Connector_Coaxial:SMA_Amphenol_132289_EdgeMount, B.Cu at (139.0, 141.6)
- added J7: XT-60, kicad-egglib:XT60PW-M, F.Cu at (113.0, 135.0)
- added J8: SERVO, Connector_PinHeader_2.54mm:PinHeader_1x03_P2.54mm_Vertical, F.Cu at (153.0, 132.0)
- added J9: SERVO, Connector_PinHeader_2.54mm:PinHeader_1x03_P2.54mm_Vertical, F.Cu at (153.0, 127.0)
- added JP1: VSEL, Jumper:SolderJumper-3_P1.3mm_Open_Pad1.0x1.5mm, F.Cu at (152.0, 101.0)
- added L1: 4.7uH, Inductor_SMD:L_1210_3225Metric, F.Cu at (121.0, 108.0)
- added Q1: DMG3402L, Package_TO_SOT_SMD:SOT-23-3, B.Cu at (109.0, 68.0)
- added Q10: DMG3402L, Package_TO_SOT_SMD:SOT-23-3, F.Cu at (109.0, 92.5)
- added Q11: DMP3099L, Package_TO_SOT_SMD:SOT-23-3, F.Cu at (109.0, 88.0)
- added Q2: DMG3402L, Package_TO_SOT_SMD:SOT-23-3, F.Cu at (109.0, 68.0)
- added Q3: DMG3402L, Package_TO_SOT_SMD:SOT-23-3, B.Cu at (109.0, 73.0)
- added Q4: DMG3402L, Package_TO_SOT_SMD:SOT-23-3, F.Cu at (109.0, 73.0)
- added Q5: DMG3402L, Package_TO_SOT_SMD:SOT-23-3, B.Cu at (109.0, 78.0)
- added Q6: DMG3402L, Package_TO_SOT_SMD:SOT-23-3, F.Cu at (109.0, 78.0)
- added Q7: DMG3402L, Package_TO_SOT_SMD:SOT-23-3, B.Cu at (109.0, 83.0)
- added Q8: DMG3402L, Package_TO_SOT_SMD:SOT-23-3, F.Cu at (109.0, 83.0)
- added Q9: DMP3099L, Package_TO_SOT_SMD:SOT-23-3, F.Cu at (109.0, 97.0)
- added R1: 5.1k, kicad-egglib:0402_1005M, F.Cu at (135.5, 55.0)
- added R10: 3.3K, kicad-egglib:0402_1005M, F.Cu at (114.0, 59.5)
- added R11: 100k, kicad-egglib:0402_1005M, B.Cu at (124.5, 98.8)
- added R12: 100k, kicad-egglib:0402_1005M, B.Cu at (121.8, 94.0)
- added R13: 100k, kicad-egglib:0402_1005M, B.Cu at (128.2, 95.5)
- added R14: 100k, kicad-egglib:0402_1005M, F.Cu at (117.0, 116.0)
- added R15: 100k, kicad-egglib:0402_1005M, F.Cu at (125.5, 54.5)
- added R16: 100k, kicad-egglib:0402_1005M, B.Cu at (135.8, 67.0)
- added R17: 100k, kicad-egglib:0402_1005M, F.Cu at (133.0, 122.0)
- added R18: 1k, kicad-egglib:0402_1005M, B.Cu at (118.8, 89.0)
- added R19: 1k, kicad-egglib:0402_1005M, B.Cu at (117.5, 89.0)
- added R2: 5.1k, kicad-egglib:0402_1005M, F.Cu at (140.5, 55.0)
- added R20: 100k, kicad-egglib:0402_1005M, B.Cu at (135.2, 75.8)
- added R21: 10k, kicad-egglib:0402_1005M, B.Cu at (111.8, 68.5)
- added R22: 1k, kicad-egglib:0402_1005M, F.Cu at (108.0, 65.5)
- added R23: 10k, kicad-egglib:0402_1005M, F.Cu at (110.0, 65.5)
- added R24: 10k, kicad-egglib:0402_1005M, F.Cu at (111.8, 68.5)
- added R25: 10k, kicad-egglib:0402_1005M, B.Cu at (111.8, 73.5)
- added R26: 10k, kicad-egglib:0402_1005M, F.Cu at (113.0, 108.5)
- added R27: 1k, kicad-egglib:0402_1005M, F.Cu at (108.0, 70.5)
- added R28: 1k, kicad-egglib:0402_1005M, F.Cu at (102.0, 107.8)
- added R29: 1k, kicad-egglib:0402_1005M, F.Cu at (108.0, 107.8)
- added R3: 33k, kicad-egglib:0402_1005M, B.Cu at (137.8, 69.2)
- added R30: 3.3k, kicad-egglib:0402_1005M, F.Cu at (113.0, 106.5)
- added R31: 10k, kicad-egglib:0402_1005M, F.Cu at (110.0, 70.5)
- added R32: 10k, kicad-egglib:0402_1005M, F.Cu at (111.8, 73.5)
- added R33: 10k, kicad-egglib:0402_1005M, B.Cu at (111.8, 78.5)
- added R34: 1k, kicad-egglib:0402_1005M, F.Cu at (108.0, 75.5)
- added R35: 10k, kicad-egglib:0402_1005M, F.Cu at (110.0, 75.5)
- added R36: 10k, kicad-egglib:0402_1005M, F.Cu at (111.8, 78.5)
- added R37: 10k, kicad-egglib:0402_1005M, B.Cu at (111.8, 83.5)
- added R38: 1k, kicad-egglib:0402_1005M, F.Cu at (108.0, 80.5)
- added R39: 10k, kicad-egglib:0402_1005M, F.Cu at (110.0, 80.5)
- added R4: 100k, kicad-egglib:0402_1005M, F.Cu at (142.8, 56.0)
- added R40: 10k, kicad-egglib:0402_1005M, F.Cu at (111.5, 96.5)
- added R41: 10k, kicad-egglib:0402_1005M, F.Cu at (111.8, 83.5)
- added R42: 10k, kicad-egglib:0402_1005M, F.Cu at (111.5, 92.0)
- added R43: 10k, kicad-egglib:0402_1005M, F.Cu at (106.5, 97.5)
- added R44: 10k, kicad-egglib:0402_1005M, F.Cu at (111.5, 86.2)
- added R5: 82k, kicad-egglib:0402_1005M, B.Cu at (138.8, 69.2)
- added R6: 1k, kicad-egglib:0402_1005M, F.Cu at (139.2, 95.0)
- added R7: 1k, kicad-egglib:0402_1005M, F.Cu at (139.2, 93.5)
- added R8: 1k, kicad-egglib:0402_1005M, F.Cu at (139.2, 92.0)
- added R9: 1k, kicad-egglib:0402_1005M, F.Cu at (139.2, 90.5)
- added REF**: MountingHole_3.2mm_M3_Pad_Via, MountingHole:MountingHole_3.2mm_M3_Pad_Via, F.Cu at (150.0, 140.0)
- added REF**: MountingHole_3.2mm_M3_Pad_Via, MountingHole:MountingHole_3.2mm_M3_Pad_Via, F.Cu at (100.0, 50.0)
- added REF**: MountingHole_3.2mm_M3_Pad_Via, MountingHole:MountingHole_3.2mm_M3_Pad_Via, F.Cu at (150.0, 50.0)
- added REF**: MountingHole_3.2mm_M3_Pad_Via, MountingHole:MountingHole_3.2mm_M3_Pad_Via, F.Cu at (100.0, 140.0)
- added REF**: Axis1, kicad-egglib:Axis1, F.Cu at (132.0, 97.0)
- added U1: USBLC6-2SC6, Package_TO_SOT_SMD:SOT-23-6, F.Cu at (138.0, 56.0)
- added U10: MLX90395KDC, Package_SO:SOIC-8_3.9x4.9mm_P1.27mm, F.Cu at (117.0, 89.0)
- added U11: W25N01GVZEIG, Package_SON:WSON-8-1EP_8x6mm_P1.27mm_EP3.4x4.3mm, B.Cu at (130.0, 77.0)
- added U12: LDL1117, Package_TO_SOT_SMD:SOT-223-3_TabPin2, F.Cu at (145.0, 100.0)
- added U13: AP62200WU, Package_TO_SOT_SMD:SOT-23-6, F.Cu at (116.0, 108.0)
- added U14: INA260, Package_SO:TSSOP-16_4.4x5mm_P0.65mm, F.Cu at (105.0, 104.0)
- added U15: SN74LVC1T45DBV, Package_TO_SOT_SMD:SOT-23-6, F.Cu at (140.5, 132.0)
- added U16: SN74LVC1T45DBV, Package_TO_SOT_SMD:SOT-23-6, F.Cu at (140.5, 127.0)
- added U17: SN74LVC1T45DBV, Package_TO_SOT_SMD:SOT-23-6, F.Cu at (140.5, 122.0)
- added U18: SN74LVC1T45DBV, Package_TO_SOT_SMD:SOT-23-6, F.Cu at (140.5, 117.0)
- added U19: SN74LVC1T45DBV, Package_TO_SOT_SMD:SOT-23-6, F.Cu at (140.5, 112.0)
- added U2: STM32F765ZGT7, Package_QFP:LQFP-144_20x20mm_P0.5mm, F.Cu at (130.0, 74.0)
- added U20: SN74LVC1T45DBV, Package_TO_SOT_SMD:SOT-23-6, F.Cu at (140.5, 107.0)
- added U3: BMI088, kicad-egglib:BMI088, F.Cu at (125.0, 95.0)
- added U4: H3LIS331DL, Package_LGA:LGA-16_3x3mm_P0.5mm_LayoutBorder3x5y, F.Cu at (125.0, 102.0)
- added U5: RFM95W-915S2, kicad-egglib:RFM9xW-xxxS2, B.Cu at (112.0, 115.0)
- added U6: ZOE-M8Q, kicad-egglib:ZOE-M8Q, F.Cu at (109.0, 56.0)
- added U7: MS560702BA03-50, kicad-egglib:MS5607-02BA, F.Cu at (125.0, 51.0)
- added U8: W25N01GVZEIG, Package_SON:WSON-8-1EP_8x6mm_P1.27mm_EP3.4x4.3mm, B.Cu at (130.0, 69.0)
- added U9: RFM96W-433S2, kicad-egglib:RFM9xW-xxxS2, B.Cu at (132.0, 127.0)
- added Y1: 48MHz, Crystal:Crystal_SMD_2520-4Pin_2.5x2.0mm, B.Cu at (116.2, 75.5)
- added Y2: 32.768kHz, Crystal:Crystal_SMD_MicroCrystal_CM9V-T1A-2Pin_1.6x1.0mm, F.Cu at (110.0, 59.8)
Routing:
- net +3.3V: track 0.00 -> 105.5 mm, vias 0 -> 78
- net SERVO0: track 0.00 -> 63.9 mm, vias 0 -> 2
- net SERVO1: track 0.00 -> 59.4 mm, vias 0 -> 2
- net +BATT: track 0.00 -> 55.6 mm, vias 0 -> 11
- net SERVO2: track 0.00 -> 55.0 mm, vias 0 -> 2
- net COM1_D1: track 0.00 -> 54.8 mm, vias 0 -> 3
- net COM1_D0: track 0.00 -> 54.4 mm, vias 0 -> 3
- net SERVO4: track 0.00 -> 52.2 mm, vias 0 -> 2
- net COM_SCK: track 0.00 -> 51.7 mm, vias 0 -> 3
- net SERVO3: track 0.00 -> 50.4 mm, vias 0 -> 2
- net COM_MOSI: track 0.00 -> 49.6 mm, vias 0 -> 3
- net Net-(JP1-C): track 0.00 -> 49.0 mm
- net PWR_SDA: track 0.00 -> 48.7 mm, vias 0 -> 2
- net PWR_SCL: track 0.00 -> 47.9 mm, vias 0 -> 2
- net SERVO5: track 0.00 -> 47.7 mm, vias 0 -> 2
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- added copper zone on F.Cu, net +3.3V
- added copper zone on In2.Cu, net +3.3V
- added copper zone on F.Cu, net +BATT
- added copper zone on In3.Cu, net +BATT
- added copper zone on F.Cu, net +VSW
- added copper zone on In3.Cu, net +VSW
- added copper zone on B.Cu, net GND
- added copper zone on F.Cu, net GND
- added copper zone on In1.Cu, net GND
- added copper zone on In4.Cu, net GND
- added copper zone on F.Cu, net Net-(D7-K)
- added copper zone on F.Cu, net Net-(J12-Pin_11)
- added copper zone on In3.Cu, net Net-(J12-Pin_11)
- added copper zone on F.Cu, net Net-(U13-SW)
- added copper zone on In3.Cu, net VBUS
Other:
- board outline added: 60 x 100 mm
- board text added: "+"
- board text added: "-"
- board text added: "0"
- board text added: "1"
- board text added: "2"
- board text added: "3"
- board text added: "3.3V"
- board text added: "4"
- board text added: "5"
- board text added: "COMMAND"
- board text added: "GND"
- board text added: "GNSS"
- board text added: "IO0"
- board text added: "IO1"
- board text added: "IO2"
- board text added: "IO3"
- board text added: "IO4"
- board text added: "IO5"
- board text added: "IO6"
- board text added: "IO7"
- board text added: "POWER"
- board text added: "POWER IN 18V MAX"
- board text added: "PYRO0"
- board text added: "PYRO1"
- board text added: "PYRO2"
- board text added: "PYRO3"
- board text added: "S"
- board text added: "TELEM"
- board text added: "VBAT"
- board text added: "~{EN}"

Commit message: Rev. 2
Parts:
- removed R13: 100k, kicad-egglib:0402_1005M
- added C55: 10uF, kicad-egglib:0805_2012M, F.Cu at (145.8, 53.0)
- added C56: 100nF, kicad-egglib:0402_1005M, F.Cu at (145.2, 59.5)
- added C57: 4.7uF, kicad-egglib:0402_1005M, F.Cu at (128.2, 97.0)
- added C58: 4.7uF, kicad-egglib:0402_1005M, F.Cu at (146.5, 59.5)
- C12, C13, C14, C21, C22, C27, C28, C36, J5, R11, R12, R18, R19, U5: moved to F.Cu
- C35, R17: moved to B.Cu
- J10, J11, J13, J14, J8, J9: footprint Connector_PinHeader_2.54mm:PinHeader_1x03_P2.54mm_Vertical -> Connector_JST:JST_XH_B3B-XH-A_1x03_P2.50mm_Vertical
- R10: value 3.3K -> 3.3k
- U10: value MLX90395KDC -> MMC5983MA; footprint Package_SO:SOIC-8_3.9x4.9mm_P1.27mm -> Package_LGA:LGA-16_3x3mm_P0.5mm
- U2: value STM32F765ZGT7 -> STM32H733ZGT6
- U3: value BMI088 -> ASM330LHB; footprint kicad-egglib:BMI088 -> Package_LGA:LGA-14_3x2.5mm_P0.5mm_LayoutBorder3x4y
- moved J2 49.0 mm to (100.0, 58.0), turned to 0 degrees
- moved C36 45.8 mm to (142.5, 55.8)
- moved U10 43.2 mm to (145.5, 56.5), turned to 90 degrees
- moved R19 40.4 mm to (142.5, 57.2), turned to 0 degrees
- moved R18 38.3 mm to (143.2, 59.5)
- moved C17 38.2 mm to (106.0, 62.0)
- moved R4 38.2 mm to (105.0, 62.0)
- moved C32 30.1 mm to (125.0, 138.5), turned to -90 degrees
- moved J5 27.1 mm to (117.0, 141.6), turned to -90 degrees
- moved C44 23.0 mm to (129.5, 102.0), turned to 180 degrees
- moved JP1 18.5 mm to (133.5, 102.0), turned to 0 degrees
- moved J7 17.2 mm to (105.5, 119.5), turned to 90 degrees
- moved REF** 17.1 mm to (115.0, 95.0)
- moved U5 17.0 mm to (124.0, 127.0), turned to -90 degrees
- moved U12 15.4 mm to (132.5, 109.0), turned to 90 degrees
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Connections:
- J7 pad 1: Net-(J12-Pin_11) -> GND
- J7 pad 2: GND -> Net-(J12-Pin_11)
- R12 pad 2: ACC_~{CS} -> IMU_~{CS}
- U10 pad 2: MAG_SDA -> +3.3V
- U10 pad 3: GND -> unconnected-(U10-Pad3)
- U10 pad 4: MAG_INT -> unconnected-(U10-Pad4)
- U10 pad 5: GND -> unconnected-(U10-Pad5)
- U10 pad 6: GND -> unconnected-(U10-Pad6)
- U10 pad 7: +3.3V -> unconnected-(U10-Pad7)
- U10 pad 8: +3.3V -> unconnected-(U10-Pad8)
- U2 pad 26: unconnected-(U2D-PC0-Pad26) -> ~{ENABLE}
- U2 pad 27: unconnected-(U2D-PC1-Pad27) -> PYRO_EN
- U2 pad 35: ~{ENABLE} -> COM1_D1
- U2 pad 36: PYRO_EN -> COM1_D0
- U2 pad 37: COM0_D1 -> COM0_D0
- U2 pad 40: COM0_D0 -> COM0_D1
- U2 pad 44: COM0_~{CS} -> COM0_~{RST}
- U2 pad 45: COM0_~{RST} -> COM0_~{CS}
- U2 pad 46: COM1_D1 -> COM1_~{CS}
- U2 pad 47: COM1_D0 -> COM1_~{RST}
- U2 pad 48: COM1_~{CS} -> unconnected-(U2C-PB2-Pad48)
- U2 pad 49: COM1_~{RST} -> unconnected-(U2E-PF11-Pad49)
- U2 pad 59: ACC_~{CS} -> unconnected-(U2E-PE8-Pad59)
- U2 pad 60: ACC_INT -> unconnected-(U2E-PE9-Pad60)
- U2 pad 63: GYR_INT -> IMU_INT1
- U2 pad 64: GYR_~{CS} -> IMU_INT2
- U2 pad 68: unconnected-(U2E-PE15-Pad68) -> IMU_~{CS}
- U3 pad 1: unconnected-(U3-INT2-Pad1) -> IMU_MISO
- U3 pad 10: IMU_MISO -> unconnected-(U3-Pad10)
- U3 pad 11: +3.3V -> unconnected-(U3-Pad11)
- U3 pad 12: GYR_INT -> IMU_~{CS}
- U3 pad 13: unconnected-(U3-INT4-Pad13) -> IMU_SCK
- U3 pad 14: ACC_~{CS} -> IMU_MOSI
- U3 pad 2: unconnected-(U3-Pad2) -> GND
- U3 pad 3: +3.3V -> GND
- U3 pad 4: GND -> IMU_INT1
- U3 pad 5: GYR_~{CS} -> +3.3V
- U3 pad 6: GND -> unconnected-(U3-Pad6)
- U3 pad 8: IMU_SCK -> +3.3V
- U3 pad 9: IMU_MOSI -> IMU_INT2
- Y1 pad 2: +3.3V -> GND
- Y1 pad 4: GND -> +3.3V
Routing:
- net MCU_SWDIO: track 11.9 -> 50.1 mm, vias 0 -> 2
- net MCU_SWCLK: track 11.4 -> 43.7 mm, vias 0 -> 2
- net COM0_D1: track 35.6 -> 58.8 mm, vias 1 -> 2
- net IMU_INT1: track 0.00 -> 21.5 mm
- net +BATT: track 55.6 -> 35.7 mm
- net GYR_INT: track 19.2 -> 0.00 mm
- net IMU_~{CS}: track 0.00 -> 19.1 mm
- net COM0_D0: track 38.2 -> 56.9 mm, vias 1 -> 2
- net ACC_~{CS}: track 18.7 -> 0.00 mm, vias 1 -> 0
- net GYR_~{CS}: track 18.5 -> 0.00 mm, vias 1 -> 0
- net IMU_INT2: track 0.00 -> 17.3 mm, vias 0 -> 2
- net MCU_~{RST}: track 44.6 -> 28.5 mm
- net ACC_INT: track 15.3 -> 0.00 mm
- net MAG_SCL: track 20.7 -> 34.5 mm, vias 1 -> 2
- net MAG_INT: track 21.5 -> 34.9 mm, vias 0 -> 2
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Other:
- board text added: "COMMAND 915 MHz"
- board text added: "EVE Flight Computer Rev. 2 Aug 2024"
- board text added: "TELEMETRY 433 MHz"
- board text removed: "COMMAND"
- board text removed: "TELEM"
